Commit message: feat: enhance README, add Gazebo configuration, and implement launch script for simulation

File: description/robot.urdf.xacro (robot description, xacro)
@@ -1,5 +1,5 @@
 <?xml version="1.0"?>
 <robot xmlns:xacro="http://www.ros.org/wiki/xacro"  name="robot">
-    <!-- Example link -->
     <xacro:include filename="robot_core.xacro" />
+    <xacro:include filename="gazebo_control.xacro" />
 </robot>

File: description/robot_core.xacro (robot description, xacro)
@@ -41,4 +41,7 @@
         </xacro:inertial_box>
     </link>
+    <gazebo reference="chassis">
+       <material>Gazebo/White</material>
+    </gazebo>
     <!-- left_wheel_joint -->
     <joint name="left_wheel_joint" type="continuous">
@@ -47,4 +50,5 @@
         <origin xyz="0 0.175 0" rpy="-${pi/2} 0 0"/>
         <axis xyz="0 0 1"/>
+        <limit effort="100.0" velocity="10.0"/>
     </joint>
     <link name="left_wheel">
@@ -64,4 +68,7 @@
         </xacro:inertial_cylinder>
     </link>
+      <gazebo reference="left_wheel">
+       <material>Gazebo/Blue</material>
+    </gazebo>
      <!-- right_wheel_joint -->
     <joint name="right_wheel_joint" type="continuous">
@@ -70,4 +77,5 @@
         <origin xyz="0 -0.175 0" rpy="${pi/2} 0 0"/>
         <axis xyz="0 0 -1"/>
+        <limit effort="100.0" velocity="10.0"/>
     </joint>
     <link name="right_wheel">
@@ -87,4 +95,7 @@
         </xacro:inertial_cylinder>
     </link>
+      <gazebo reference="right_wheel">
+       <material>Gazebo/Blue</material>
+    </gazebo>
  <!-- caster_wheel_joint -->
     <joint name="caster_wheel_joint" type="fixed">
@@ -109,3 +120,8 @@
         </xacro:inertial_sphere>
     </link>
+      <gazebo reference="caster_wheel">
+       <material>Gazebo/Black</material>
+       <mu1 value="0.001" />
+       <mu2 value="0.001" />
+    </gazebo>
 </robot>
