Commit message: feat: add slam toolbox launch configuration, update README with usage instructions, and enhance robot description with base footprint link

File: description/robot_core.xacro (robot description, xacro)
@@ -16,4 +16,11 @@
 <!-- Base link -->
     <link name="base_link">
+    </link>
+    <joint name="base_footprint_link" type="fixed">
+        <parent link="base_link"/>
+        <child link="base_footprint"/>
+        <origin xyz="0 0 0" rpy="0 0 0"/>
+    </joint>
+    <link name="base_footprint">
     </link>
 <!-- Chassis link-->
